Commit message: Fixed the parameters' bugs in ros_arduino_bridge

File: src/mycar_description/urdf/car_base.urdf.xacro (robot description, xacro)
@@ -8,7 +8,7 @@
         </visual>
     </link>
-    <xacro:property name="base_radius" value="0.12" />
-    <xacro:property name="base_length" value="0.12" />
-    <xacro:property name="lidi" value="0.01" />
+    <xacro:property name="base_radius" value="0.18" />
+    <xacro:property name="base_length" value="0.22" />
+    <xacro:property name="lidi" value="0.02" />
     <xacro:property name="base_joint_z" value="${base_length / 2 + lidi}" />
     <link name="base_link">
@@ -28,6 +28,6 @@
         <origin xyz="0 0 ${base_joint_z}" rpy="0 0 0" />
     </joint>
-    <xacro:property name="wheel_radius" value="0.029" />
-    <xacro:property name="wheel_length" value="0.025" />
+    <xacro:property name="wheel_radius" value="0.05" />
+    <xacro:property name="wheel_length" value="0.04" />
     <xacro:property name="PI" value="3.1415927" />
     <xacro:property name="wheel_joint_z" value="${(base_length / 2 + lidi - wheel_radius) * -1}" />

File: src/mycar_description/urdf/car_camera.urdf.xacro (robot description, xacro)
@@ -3,5 +3,5 @@
     <xacro:property name="camera_width" value="0.05" />
     <xacro:property name="camera_height" value="0.04" />
-    <xacro:property name="joint_camera_x" value="0.1" />
+    <xacro:property name="joint_camera_x" value="0.165" />
     <xacro:property name="joint_camera_y" value="0" />
     <xacro:property name="joint_camera_z" value="${(base_length / 2) + (camera_height / 2)}" />

File: src/mycar_description/urdf/car_laser.urdf.xacro (robot description, xacro)
@@ -1,7 +1,7 @@
 <robot name="mycar" xmlns:xacro="http://wiki.ros.org/xacro">
-    <xacro:property name="support_radius" value="0.01" />
-    <xacro:property name="support_length" value="0.14" />
-    <xacro:property name="laser_radius" value="0.08" />
-    <xacro:property name="laser_length" value="0.03" />
+    <xacro:property name="support_radius" value="0.05" />
+    <xacro:property name="support_length" value="0.03" />
+    <xacro:property name="laser_radius" value="0.035" />
+    <xacro:property name="laser_length" value="0.025" />
     <xacro:property name="joint_support_x" value="0" />
     <xacro:property name="joint_support_y" value="0" />
@@ -30,5 +30,5 @@
                 <cylinder radius="${laser_radius}" length="${laser_length}" />
             </geometry>
-            <material name="black">
+            <material name="red">
                 <color rgba="0 0 0 0.5" />
             </material>

Commit message: Adjust the PID params with load. Nav function hasn't been finished.

File: src/mycar_description/urdf/car_base.urdf.xacro (robot description, xacro)
@@ -9,5 +9,5 @@
     </link>
     <xacro:property name="base_radius" value="0.18" />
-    <xacro:property name="base_length" value="0.22" />
+    <xacro:property name="base_length" value="0.21" />
     <xacro:property name="lidi" value="0.02" />
     <xacro:property name="base_joint_z" value="${base_length / 2 + lidi}" />

File: src/mycar_description/urdf/car_laser.urdf.xacro (robot description, xacro)
@@ -1,11 +1,11 @@
 <robot name="mycar" xmlns:xacro="http://wiki.ros.org/xacro">
     <xacro:property name="support_radius" value="0.05" />
-    <xacro:property name="support_length" value="0.03" />
+    <xacro:property name="support_length" value="0.15" />
     <xacro:property name="laser_radius" value="0.035" />
-    <xacro:property name="laser_length" value="0.025" />
+    <xacro:property name="laser_length" value="0.024" />
     <xacro:property name="joint_support_x" value="0" />
     <xacro:property name="joint_support_y" value="0" />
     <xacro:property name="joint_support_z" value="${base_length / 2 + support_length / 2}" />
-    <xacro:property name="joint_laser_x" value="-0.03" />
+    <xacro:property name="joint_laser_x" value="0.0" />
     <xacro:property name="joint_laser_y" value="0.0" />
     <xacro:property name="joint_laser_z" value="${support_length / 2 + laser_length / 2}" />
