Commit message: Finished the move_base function and nav parameters

File: src/mycar_description/urdf/car_camera.urdf.xacro (robot description, xacro)
@@ -1,7 +1,7 @@
 <robot name="mycar" xmlns:xacro="http://wiki.ros.org/xacro">
-    <xacro:property name="camera_length" value="0.02" />
+    <xacro:property name="camera_length" value="0.03" />
     <xacro:property name="camera_width" value="0.05" />
-    <xacro:property name="camera_height" value="0.05" />
-    <xacro:property name="joint_camera_x" value="0.08" />
+    <xacro:property name="camera_height" value="0.04" />
+    <xacro:property name="joint_camera_x" value="0.1" />
     <xacro:property name="joint_camera_y" value="0" />
     <xacro:property name="joint_camera_z" value="${(base_length / 2) + (camera_height / 2)}" />

File: src/mycar_description/urdf/car_laser.urdf.xacro (robot description, xacro)
@@ -1,13 +1,13 @@
 <robot name="mycar" xmlns:xacro="http://wiki.ros.org/xacro">
     <xacro:property name="support_radius" value="0.01" />
-    <xacro:property name="support_length" value="0.15" />
-    <xacro:property name="laser_radius" value="0.03" />
-    <xacro:property name="laser_length" value="0.05" />
+    <xacro:property name="support_length" value="0.14" />
+    <xacro:property name="laser_radius" value="0.08" />
+    <xacro:property name="laser_length" value="0.03" />
     <xacro:property name="joint_support_x" value="0" />
     <xacro:property name="joint_support_y" value="0" />
     <xacro:property name="joint_support_z" value="${base_length / 2 + support_length / 2}" />
-    <xacro:property name="joint_laser_x" value="0" />
-    <xacro:property name="joint_laser_y" value="0" />
-    <xacro:property name="joint_laser_z" value="${support_length / 2 + laser_length / 2}" />
+    <xacro:property name="joint_laser_x" value="-0.03" />
+    <xacro:property name="joint_laser_y" value="-0.03" />
+    <xacro:property name="joint_laser_z" value="${support_length / 2 + laser_length / 2 + 0.26}" />
     <link name="support">
         <visual>

Commit message: Found out the rr_auto_dock is not realiable. A new method has been introduced.

File: src/mycar_description/urdf/car_camera.urdf.xacro (robot description, xacro)
@@ -20,5 +20,5 @@
         <parent link="base_link" />
         <child link="camera" />
-        <origin xyz="${joint_camera_x} ${joint_camera_y} ${joint_camera_z}" rpy="0 0 0" />
+        <origin xyz="${joint_camera_x} ${joint_camera_y} ${joint_camera_z}" rpy="-1.309 0 -1.57" />
     </joint>
 </robot>

Commit message: modified the behavoirs_tree's parameters and logics with physical dock requirement

File: src/mycar_description/urdf/car_camera.urdf.xacro (robot description, xacro)
@@ -20,5 +20,6 @@
         <parent link="base_link" />
         <child link="camera" />
-        <origin xyz="${joint_camera_x} ${joint_camera_y} ${joint_camera_z}" rpy="-1.309 0 -1.57" />
+        <!-- <origin xyz="${joint_camera_x} ${joint_camera_y} ${joint_camera_z}" rpy="-1.309 0 -1.57" /> -->
+        <origin xyz="${joint_camera_x} ${joint_camera_y} ${joint_camera_z}" rpy="-1.57 0 -1.57" />
     </joint>
 </robot>

Commit message: Modified the code of visiual_docking part. Image freeze problem hasn't been solved.

File: src/mycar_description/urdf/car_camera.urdf.xacro (robot description, xacro)
@@ -1,7 +1,7 @@
 <robot name="mycar" xmlns:xacro="http://wiki.ros.org/xacro">
-    <xacro:property name="camera_length" value="0.03" />
+    <xacro:property name="camera_length" value="0.06" />
     <xacro:property name="camera_width" value="0.05" />
-    <xacro:property name="camera_height" value="0.04" />
-    <xacro:property name="joint_camera_x" value="0.165" />
+    <xacro:property name="camera_height" value="0.09" />
+    <xacro:property name="joint_camera_x" value="0.127" />
     <xacro:property name="joint_camera_y" value="0" />
     <xacro:property name="joint_camera_z" value="${(base_length / 2) + (camera_height / 2)}" />
@@ -21,5 +21,5 @@
         <child link="camera" />
         <!-- <origin xyz="${joint_camera_x} ${joint_camera_y} ${joint_camera_z}" rpy="-1.309 0 -1.57" /> -->
-        <origin xyz="${joint_camera_x} ${joint_camera_y} ${joint_camera_z}" rpy="-1.57 0 -1.57" />
+        <origin xyz="${joint_camera_x} ${joint_camera_y} ${joint_camera_z}" rpy="0 0 0" />
     </joint>
 </robot>

Commit message: Finished modifing camera_vision function.

File: src/mycar_description/urdf/car_camera.urdf.xacro (robot description, xacro)
@@ -1,5 +1,5 @@
 <robot name="mycar" xmlns:xacro="http://wiki.ros.org/xacro">
-    <xacro:property name="camera_length" value="0.06" />
-    <xacro:property name="camera_width" value="0.05" />
+    <xacro:property name="camera_length" value="0.05" />
+    <xacro:property name="camera_width" value="0.06" />
     <xacro:property name="camera_height" value="0.09" />
     <xacro:property name="joint_camera_x" value="0.127" />
@@ -20,6 +20,6 @@
         <parent link="base_link" />
         <child link="camera" />
-        <!-- <origin xyz="${joint_camera_x} ${joint_camera_y} ${joint_camera_z}" rpy="-1.309 0 -1.57" /> -->
-        <origin xyz="${joint_camera_x} ${joint_camera_y} ${joint_camera_z}" rpy="0 0 0" />
+        <!-- <origin xyz="${joint_camera_x} ${joint_camera_y} ${joint_camera_z}" rpy="-1.57 0 -1.57" /> -->
+        <origin xyz="${joint_camera_x} ${joint_camera_y} ${joint_camera_z}" rpy="-1.57 0 -1.57" />
     </joint>
 </robot>
